File: kimchi_ulid.sch (KiCad schematic (older format))
At the start: 8 parts, among them J1 DF40HC(3.5)-60DS, J2 DF40HC(3.5)-60DS, U1 24C32

Commit message: Updates for 0.92 version
Parts:
- added D1: PMEG1020EH, Diode_SMD:D_SOD-123F, symbol Diode:PMEG1020EH
- added K1: KIMCHI_MICRO, kimchi_ulid:KIMCHI_MICRO, symbol kimchi_ulid:KIMCHI_MICRO
- H1, H2, H3, H4: footprint kimchi_ulid:MountingHole_3mm_Pad -> kimchi_ulid:MountingHole_M2_Standoff; Mfgr (none) -> Würth; Mfgrpart (none) -> 9774035943R
Connections:
- net UIM_DATA is gone; now on net VCHG: J1.55 (Pin_55)
- net UIM_PWR is gone; now on net VCHG: J1.56 (Pin_56)
- net UIM_RESET_N is gone; now on net VCHG: J1.53 (Pin_53)
- net UIM_VPP is gone; now on net VCHG: J1.52 (Pin_52)
- net GND: no longer J1.11 (Pin_11), J1.51 (Pin_51)
- net VDD_1V8: no longer J2.42 (Pin_42)
- net VDD_3V3: no longer J2.54 (Pin_54)
- net UIM_CLK renamed VCHG
- net VCHG: now also D1.1 (K)
- new net VCHG_PROT: D1.2 (A)
- no-connect marks 0 -> 5
Other:
- note added: "0.9A max"
- note added: "1.2A max"
- note added: "1.5A max"
- note added: "EEPROM for lid identification (if needed)\nExpected on I2C4 @ 7-bit 0x57"
- note added: "Prevent VCHG backfeed (if needed)\nVCHG 4.5 - 6V OK\nE.G. PMEG1020 Vf=460mV @ 2A"
- note added: "Recommend standoffs populated on lid\nMatch height of J1/J2 (typ. 3.5 mm)\nWürth WA-SMST 9774035943R (non-threaded)\nWürth WA-SMSI 9774035243R (threaded)"
- moved on the sheet: H1, H2, H3, H4, U1
