File: kimchi_ulid.kicad_pcb (KiCad board)
At the start: 4 copper layers, 65 x 32 mm, 8 parts, among them J1 DF40HC(3.5)-60DS, J2 DF40HC(3.5)-60DS, U1 24C32

Commit message: Remove user comments left over from project creation
Other:
- board text removed: "All tolerances +/-10%. Unless otherwise noted, 50 Ohm single-ended. Layer 1, Layer 4 (kimchi_ulid-F_Cu.gtl, kimchi_ulid-B_Cu.gbl) Single ended: Width: 4.79 mils Impedance: 50 Ohms Differential: Width / Gap: 4.99 mils / 4 mils Impedance: 85 Ohms Differential: Width / Gap: 3.99 mils / 3.5 mils Impedance: 90 Ohms Differential: Width / Gap: 3.39 mils / 4.1 mils Impedance: 100 Ohms Layer 2, 3 (kimchi_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"
Changed lines of the file:
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@@
-(kicad_pcb (version 20171130) (host pcbnew "(5.1.2-1)-1")
+(kicad_pcb (version 20171130) (host pcbnew "(5.1.5-0-10_14)")
   (general
     (thickness 1.6)
-    (drawings 43)
+    (drawings 42)
     (tracks 8)
     (zones 0)
@@
   )
   (setup
-    (last_trace_width 0.0762)
+    (last_trace_width 0.127)
     (user_trace_width 0.0762)
     (user_trace_width 0.0889)
@@
     (diff_pair_width 0.127)
     (diff_pair_gap 0.127)
-    (add_net /CAM_CK_N)
-    (add_net /CAM_CK_P)
-    (add_net /CAM_D0_N)
-    (add_net /CAM_D0_P)
-    (add_net /CAM_D1_N)
-    (add_net /CAM_D1_P)
-    (add_net /CAM_D2_N)
-    (add_net /CAM_D2_P)
-    (add_net /CAM_D3_N)
-    (add_net /CAM_D3_P)
-    (add_net /DISP_CK_N)
-    (add_net /DISP_CK_P)
-    (add_net /DISP_D0_N)
-    (add_net /DISP_D0_P)
-    (add_net /DISP_D1_N)
-    (add_net /DISP_D1_P)
-    (add_net /DISP_D2_N)
-    (add_net /DISP_D2_P)
-    (add_net /DISP_D3_N)
-    (add_net /DISP_D3_P)
-    (add_net /ENET_MDC)
-    (add_net /ENET_MDIO)
-    (add_net /ENET_RD0)
-    (add_net /ENET_RD1)
-    (add_net /ENET_RD2)
-    (add_net /ENET_RD3)
-    (add_net /ENET_RXC)
-    (add_net /ENET_RX_CTL)
-    (add_net /ENET_TD0)
-    (add_net /ENET_TD1)
-    (add_net /ENET_TD2)
-    (add_net /ENET_TD3)
-    (add_net /ENET_TXC)
-    (add_net /ENET_TX_CTL)
-    (add_net /USDHC3_CLK)
-    (add_net /USDHC3_CMD)
-    (add_net /USDHC3_DATA0)
-    (add_net /USDHC3_DATA1)
-    (add_net /USDHC3_DATA2)
-    (add_net /USDHC3_DATA3)
-    (add_net ECSPI1_MISO)
-    (add_net ECSPI1_MOSI)
-    (add_net ECSPI1_SCLK)
-    (add_net ECSPI1_SS0)
-    (add_net ECSPI2_MISO)
-    (add_net ECSPI2_MOSI)
-    (add_net ECSPI2_SCLK)
-    (add_net ECSPI2_SS0)
     (add_net GND)
-    (add_net GPIO1[0])
-    (add_net GPIO1[10])
-    (add_net GPIO1[11])
-    (add_net GPIO1[12])
-    (add_net GPIO1[13])
-    (add_net GPIO1[14])
-    (add_net GPIO1[15])
-    (add_net GPIO1[1])
-    (add_net GPIO1[9])
-    (add_net I2C1_SCL)
-    (add_net I2C1_SDA)
-    (add_net I2C2_SCL)
-    (add_net I2C2_SDA)
-    (add_net I2C3_SCL)
-    (add_net I2C3_SDA)
     (add_net I2C4_SCL)
     (add_net I2C4_SDA)
-    (add_net "Net-(J2-Pad58)")
-    (add_net PCIE_USB_D_N)
-    (add_net PCIE_USB_D_P)
-    (add_net SAI2_MCLK)
-    (add_net SAI2_RXC)
-    (add_net SAI2_RXD0)
-    (add_net SAI2_RXFS)
-    (add_net SAI2_TXC)
-    (add_net SAI2_TXD0)
-    (add_net SAI2_TXFS)
-    (add_net SAI3_MCLK)
-    (add_net SAI3_RXC)
-    (add_net SAI3_RXD)
-    (add_net SAI3_RXFS)
-    (add_net SAI3_TXC)
-    (add_net SAI3_TXD)
-    (add_net SAI3_TXFS)
-    (add_net UART1_RX)
-    (add_net UART1_TX)
-    (add_net UART3_RX)
-    (add_net UART3_TX)
-    (add_net UIM_CLK)
-    (add_net UIM_DATA)
-    (add_net UIM_PWR)
-    (add_net UIM_RESET_N)
-    (add_net UIM_VPP)
-    (add_net USB2_DN)
-    (add_net USB2_DP)
-    (add_net USB2_ID)
-    (add_net USB2_VBUS)
     (add_net VDD_1V8)
     (add_net VDD_3V3)
@@
     (effects (font (size 1 1) (thickness 0.15)))
   )
-  (gr_text "All tolerances +/-10%. Unless otherwise noted, 50 Ohm single-ended.\n\nLayer 1, Layer 4 (kimchi_ulid-F_Cu.gtl, kimchi_ulid-B_Cu.gbl)\n    Single ended:\n        Width: 4.79 mils\n        Impedance: 50 Ohms\n    Differential:\n        Width / Gap: 4.99 mils / 4 mils\n        Impedance: 85 Ohms\n    Differential:\n        Width / Gap: 3.99 mils / 3.5 mils\n        Impedance: 90 Ohms\n    Differential:\n        Width / Gap: 3.39 mils / 4.1 mils\n        Impedance: 100 Ohms\n\nLayer 2, 3 (kimchi_ulid-In1_Cu.g2, kimchi_ulid-In2_Cu.g3)\n    Single ended:\n        Width: 3.59 mils\n        Impedance:  50 Ohms" (at 179 111) (layer Cmts.User)
-    (effects (font (size 0.508 0.508) (thickness 0.0508)) (justify left))
-  )
   (dimension 32 (width 0.15) (layer Dwgs.User)

Commit message: Updates for 0.92 version
Parts:
- added D1: PMEG1020EH, Diode_SMD:D_SOD-123F, B.Cu at (157.0, 101.0)
- added K1: KIMCHI_MICRO, kimchi_ulid:KIMCHI_MICRO, B.Cu at (107.0, 126.0)
- H1, H2, H3, H4: footprint kimchi_ulid:MountingHole_3mm_Pad -> kimchi_ulid:MountingHole_M2_Standoff; moved to B.Cu
- moved U1 44.0 mm to (125.0, 96.0), turned to 0 degrees
Connections:
- J1 pad 11: GND -> (no net)
- J1 pad 51: GND -> (no net)
- J1 pad 52: (no net) -> VCHG
- J1 pad 53: (no net) -> VCHG
- J1 pad 54: (no net) -> VCHG
- J1 pad 55: (no net) -> VCHG
- J1 pad 56: (no net) -> VCHG
- J2 pad 42: VDD_1V8 -> (no net)
- J2 pad 54: VDD_3V3 -> (no net)
Routing:
- net VDD_3V3: track 4.95 -> 0.00 mm, vias 2 -> 0
Other:
- net class Default: clearance 0.127 -> 0.0889
- rule solder_mask_min_width: 0.1016 -> 0.2032
- rule trace_clearance: 0.127 -> 0.0889

Commit message: Set solder mask clearances to zero
Other:
- rule pad_to_mask_clearance: 0.0508 -> 0

Commit message: Update template to be compatible with kicad 9
Signed-off-by: Michael Welling <mwelling79@gmail.com>
Other:
- net class CSI/DSI removed
- net class Default removed
- net class PCIE removed
- net class USB removed
